File: koken-2026-welcome/koken-2026-welcome.kicad_sch (KiCad schematic)
At the start: 5 parts, among them J1 USB_C_Receptacle_USB2.0_16P, U1 CH32V003JxMx

Commit message: add neopixel
Parts:
- added C1, C2: 1u, symbol Device:C
- added C3, C4, C5: 100n, symbol Device:C_Small
- added D1, D2, D3: WS2812B-2020, LED_SMD:LED_WS2812B-2020_PLCC4_2.0x2.0mm, symbol LED:WS2812B-2020
- added U2: AP7333, Library:AP7333, symbol New_Library:AP7333
Connections:
- net +3.3V: now also C2.1, U2.2 (VO)
- net +5V: now also C1.1, C3.1, C4.1, C5.1, D1.4 (VDD), D2.4 (VDD), D3.4 (VDD), U2.1 (VI)
- net GND: now also C1.2, C2.2, C3.2, C4.2, C5.2, D1.2 (VSS), D2.2 (VSS), D3.2 (VSS), U2.3 (GND)
- net WS2812C: now also D1.3 (DIN)
- new net: D2.1 (DOUT), D3.3 (DIN)
- new net: D1.1 (DOUT), D2.3 (DIN)
- no-connect marks 2 -> 3
Other:
- note added: "https://github.com/cnlohr/rv003usb"
- moved on the sheet: R3, U1

Commit message: USBキーボードとNeopixel光るくん
Parts:
- added R4: 10k, symbol Device:R
- added SW1: SW_Push, symbol Switch:SW_Push
Connections:
- net GND: now also R4.1
- net KEY: now also R4.2, SW1.2
- new net 3.3v: SW1.1

Commit message: 回路図完成
Parts:
- added BT1: CR2032, symbol Device:Battery_Cell
- added J2: Conn_01x03_Pin, symbol Connector:Conn_01x03_Pin
- added SW2: SW_SPDT, symbol Switch:SW_SPDT
- C1, C2, C3, C4, C5: footprint (none) -> Capacitor_SMD:C_0603_1608Metric_Pad1.08x0.95mm_HandSolder
- R1, R2, R3, R4: footprint (none) -> Resistor_SMD:R_0603_1608Metric_Pad0.98x0.95mm_HandSolder
Connections:
- net +3.3V: now also SW2.1 (A); no longer U1.4 (VDD)
- net +5V: no longer C3.1, C4.1, C5.1, D1.4 (VDD), D2.4 (VDD), D3.4 (VDD)
- net GND: now also BT1.2 (-), J2.1 (Pin_1)
- net SWIO: now also J2.3 (Pin_3)
- net 3.3v renamed VDD
- net VDD: now also C3.1, C4.1, C5.1, D1.4 (VDD), D2.4 (VDD), D3.4 (VDD), U1.4 (VDD), J2.2 (Pin_2), SW2.2 (B)
- new net BAT: BT1.1 (+), SW2.3 (C)
Other:
- moved on the sheet: C1, C2, C3, C4, C5, D1, D2, D3, R3, R4, SW1, U1

Commit message: assign footprint
Parts:
- BT1, SW1: footprint (none) -> Library:CherryMX_Red
- J1: footprint (none) -> Connector_USB:USB_C_Receptacle_GCT_USB4105-xx-A_16P_TopMnt_Horizontal
- J2: footprint (none) -> Connector_PinHeader_2.54mm:PinHeader_1x03_P2.54mm_Vertical
- SW2: footprint (none) -> Button_Switch_THT:SW_Slide-03_Wuerth-WS-SLTV_10x2.5x6.4_P2.54mm
Changed lines of the file:
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@@
 			)
 		)
-		(property "Footprint" ""
+		(property "Footprint" "Button_Switch_THT:SW_Slide-03_Wuerth-WS-SLTV_10x2.5x6.4_P2.54mm"
 			(at 55.88 148.59 0)
 			(effects
@@
 			)
 		)
-		(property "Footprint" ""
+		(property "Footprint" "Connector_PinHeader_2.54mm:PinHeader_1x03_P2.54mm_Vertical"
 			(at 146.05 110.49 0)
 			(effects
@@
 			)
 		)
-		(property "Footprint" ""
+		(property "Footprint" "Library:CherryMX_Red"
 			(at 113.03 115.57 0)
 			(effects
@@
 			)
 		)
-		(property "Footprint" ""
+		(property "Footprint" "Connector_USB:USB_C_Receptacle_GCT_USB4105-xx-A_16P_TopMnt_Horizontal"
 			(at 58.42 87.63 0)
 			(effects
@@
 			)
 		)
-		(property "Footprint" ""
+		(property "Footprint" "Library:CherryMX_Red"
 			(at 81.28 105.156 90)
 			(effects

Commit message: fix
Parts:
- BT1: footprint Library:CherryMX_Red -> Battery:BatteryHolder_MPD_BC2003_1x2032
Connections:
- net D+: no longer U1.6 (PC2)
- net D-: now also U1.6 (PC2)
Changed lines of the file:
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@@
 		)
 	)
-	(global_label "D+"
+	(global_label "D-"
 		(shape input)
 		(at 97.79 83.82 180)
@@
 			)
 		)
-		(property "Footprint" "Library:CherryMX_Red"
+		(property "Footprint" "Battery:BatteryHolder_MPD_BC2003_1x2032"
 			(at 81.28 105.156 90)
 			(effects

Commit message: -
Parts:
- renumbered C4 to C3, C3 to C4
Changed lines of the file:
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@@
 		(dnp no)
 		(fields_autoplaced yes)
-		(property "Reference" "C4"
+		(property "Reference" "C3"
 			(at 105.41 133.3562 0)
 			(effects
@@
 			(project ""
 				(path "/c1514d4b-c430-4cc3-b61b-88eeca3cb740"
-					(reference "C4")
+					(reference "C3")
 					(unit 1)
 				)
@@
 		(dnp no)
 		(fields_autoplaced yes)
-		(property "Reference" "C3"
+		(property "Reference" "C4"
 			(at 129.54 133.3562 0)
 			(effects
@@
 			(project "koken-2026-welcome"
 				(path "/c1514d4b-c430-4cc3-b61b-88eeca3cb740"
-					(reference "C3")
-					(unit 1)
-				)
+					(reference "C4")
+					(unit 1)
+				)

Commit message: add c
Parts:
- added C6: 0.1u, symbol Device:C_Small
Connections:
- net GND: now also C6.2
- net VDD: now also C6.1
Changed lines of the file:
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@@
+	(wire
+		(pts
+			(xy 151.13 76.2) (xy 152.4 77.47)
+		)
+		(stroke
+			(width 0)
+			(type default)
+		)
+	)
+	(wire
+		(pts
+			(xy 151.13 91.44) (xy 115.57 91.44)
+		)
+		(stroke
+			(width 0)
+			(type default)
+		)
+	)
 	(wire
 		(pts
@@
 	(wire
 		(pts
+			(xy 152.4 77.47) (xy 152.4 81.28)
+		)
+		(stroke
+			(width 0)
+			(type default)
+		)
+	)
+	(wire
+		(pts
+			(xy 151.13 76.2) (xy 115.57 76.2)
+		)
+		(stroke
+			(width 0)
+			(type default)
+		)
+	)
+	(wire
+		(pts
 			(xy 69.85 85.09) (xy 69.85 87.63)
 		)
@@
 	(wire
 		(pts
+			(xy 151.13 91.44) (xy 152.4 90.17)
+		)
+		(stroke
+			(width 0)
+			(type default)
+		)
+	)
+	(wire
+		(pts
 			(xy 151.13 144.78) (xy 149.86 146.05)
 		)
@@
 		(pts
 			(xy 93.98 146.05) (xy 101.6 146.05)
+		)
+		(stroke
+			(width 0)
+			(type default)
+		)
+	)
+	(wire
+		(pts
+			(xy 152.4 90.17) (xy 152.4 86.36)
 		)
 		(stroke
@@
 					(unit 1)
 				)
+			)
+		)
+	)
+	(symbol
+		(lib_id "Device:C_Small")
+		(at 152.4 83.82 0)
+		(unit 1)
+		(exclude_from_sim no)
+		(in_bom yes)
+		(on_board yes)
+		(dnp no)
+		(fields_autoplaced yes)
+		(property "Reference" "C6"
+			(at 154.94 82.5562 0)
+			(effects
+				(font
+					(size 1.27 1.27)
+				)
+				(justify left)
+			)
+		)
+		(property "Value" "0.1u"
+			(at 154.94 85.0962 0)
+			(effects
+				(font
+					(size 1.27 1.27)
+				)
+				(justify left)
+			)
+		)
+		(property "Footprint" ""
+			(at 152.4 83.82 0)
+			(effects
+				(font
+					(size 1.27 1.27)
+				)
+				(hide yes)
+			)
+		)
+		(property "Datasheet" "~"
+			(at 152.4 83.82 0)
+			(effects
+				(font
+					(size 1.27 1.27)
+				)
+				(hide yes)
+			)
+		)
+		(property "Description" "Unpolarized capacitor, small symbol"
+			(at 152.4 83.82 0)
+			(effects
+				(font
+					(size 1.27 1.27)
+				)
+				(hide yes)
+			)
+		)
+		(pin "2"
+		)
+		(pin "1"
+		)
+		(instances
+			(project ""
+				(path "/c1514d4b-c430-4cc3-b61b-88eeca3cb740"
+					(reference "C6")
+					(unit 1)
+				)

Commit message: -
Parts:
- C6: footprint (none) -> Capacitor_SMD:C_0603_1608Metric_Pad1.08x0.95mm_HandSolder
Changed lines of the file:
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@@
 			)
 		)
-		(property "Footprint" ""
+		(property "Footprint" "Capacitor_SMD:C_0603_1608Metric_Pad1.08x0.95mm_HandSolder"
 			(at 152.4 83.82 0)
 			(effects
