File: koken-2026-welcome/koken-2026-welcome.kicad_pcb (KiCad board)
At the start: 2 copper layers, 44 x 44 mm, 21 parts, among them J1 USB_C_Receptacle_USB2.0_16P, J2 Conn_01x03_Pin, SW1 SW_Push, SW2 SW_SPDT, U1 CH32V003JxMx, U2 AP7333

Commit message: -
Parts:
- added C6: 0.1u, Capacitor_SMD:C_0603_1608Metric_Pad1.08x0.95mm_HandSolder, B.Cu at (134.0, 103.5)
- moved SW2 127.9 mm to (130.0, 107.0), turned to -90 degrees
- moved R4 85.4 mm to (134.0, 111.5), turned to 180 degrees
- moved R3 76.6 mm to (141.1, 106.7), turned to -90 degrees
- moved C2 70.2 mm to (159.8, 105.0), turned to 180 degrees
- moved U2 68.4 mm to (159.4, 101.0), turned to 180 degrees
- moved C1 67.3 mm to (159.8, 100.0), turned to 180 degrees
- moved J2 51.4 mm to (152.5, 112.0), turned to -90 degrees
- moved D1 47.8 mm to (140.4, 119.0), turned to 180 degrees
- moved C3 43.5 mm to (140.4, 121.1), turned to 180 degrees
- moved D2 40.6 mm to (150.0, 127.5), turned to 180 degrees
- moved C4 36.7 mm to (150.0, 129.6), turned to 180 degrees
- moved D3 27.2 mm to (159.9, 119.0), turned to 180 degrees
- moved C5 22.5 mm to (159.9, 121.3), turned to 180 degrees
- moved R2 9.84 mm to (166.4, 113.5)
- moved R1 8.25 mm to (166.4, 100.5)
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Routing:
- net VDD: track 0.00 -> 81.6 mm
- net BAT: track 0.00 -> 50.7 mm
- net +3.3V: track 0.00 -> 40.6 mm
- net D-: track 0.00 -> 29.4 mm
- net D+: track 0.00 -> 28.9 mm
- net KEY: track 0.00 -> 16.7 mm
- net WS2812C: track 0.00 -> 14.2 mm, vias 0 -> 1
- net Net-(D2-DOUT): track 0.00 -> 13.3 mm
- net +5V: track 0.00 -> 12.1 mm, vias 0 -> 2
- net Net-(D1-DOUT): track 0.00 -> 10.8 mm
- net SWIO: track 0.00 -> 9.91 mm
- net Net-(J1-CC1): track 0.00 -> 6.64 mm
- net Net-(J1-CC2): track 0.00 -> 6.31 mm
- net DPU: track 0.00 -> 2.49 mm
- net GND: vias 0 -> 25
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- added copper zone on B.Cu, net GND
- added copper zone on F.Cu, net GND

Commit message: pro
Co-authored-by: Mcbeeringi⁉️ <git@mcbeeringi.dev>
Parts:
- J2: moved to B.Cu
- moved R1 75.0 mm to (93.0, 85.0), turned to -90 degrees
- moved J1 73.0 mm to (100.0, 81.9), turned to 0 degrees
- moved D3 71.1 mm to (90.0, 106.0), turned to 0 degrees
- moved J2 68.7 mm to (90.0, 83.5), turned to 180 degrees
- moved R2 65.9 mm to (107.0, 85.0), turned to -90 degrees
- moved C2 58.2 mm to (103.4, 90.8)
- moved C1 57.7 mm to (103.4, 88.0)
- moved U2 54.9 mm to (106.1, 87.9)
- moved C3 53.2 mm to (90.0, 104.0)
- moved C5 52.8 mm to (110.0, 104.0)
- moved C4 52.4 mm to (100.0, 114.0)
- moved BT1 51.7 mm to (100.0, 111.0)
- moved G*** 51.7 mm to (100.0, 100.0) (x2)
- moved D2 51.3 mm to (100.0, 116.0), turned to 0 degrees
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Routing:
- net VDD: track 81.6 -> 6.54 mm, vias 0 -> 1
- net BAT: track 50.7 -> 0.00 mm, vias 0 -> 4
- net +3.3V: track 40.6 -> 0.00 mm
- net D+: track 28.9 -> 8.66 mm
- net D-: track 29.4 -> 12.1 mm
- net +5V: track 12.1 -> 0.00 mm, vias 2 -> 4
- net WS2812C: track 14.2 -> 24.8 mm
- net Net-(D1-DOUT): track 10.8 -> 15.3 mm
- net SWIO: track 9.91 -> 5.78 mm
- net GND: track 0.00 -> 2.72 mm, vias 25 -> 6
- net KEY: track 16.7 -> 15.6 mm
- net Net-(D2-DOUT): track 13.3 -> 12.7 mm
- net (no net): vias 2 -> 0
- added copper zone on B.Cu, net +3.3V
- added copper zone on B.Cu, net +5V
- added copper zone on F.Cu, net +5V
- added copper zone on F.Cu, net BAT
- added copper zone on F.Cu, net VDD
Other:
- outline, holes or cut-outs redrawn
