File: koken-2026-welcome/koken-2026-welcome.kicad_pcb (KiCad board)
At the start: 2 copper layers, 44 x 44 mm, 22 parts, among them J1 USB_C_Receptacle_USB2.0_16P, J2 Conn_01x03_Pin, SW1 SW_Push, SW2 SW_SPDT, U1 CH32V003JxMx, U2 AP7333

Commit message: -
Parts:
- added ?: https://ueckoken.club/, QRCODE, B.Cu at (119.7, 96.0)
- added H1: MountingHole, MountingHole:MountingHole_2.2mm_M2, B.Cu at (82.4, 117.6)
- BT1: footprint Battery:BatteryHolder_MPD_BC2003_1x2032 -> Battery:BatteryHolder_Multicomp_BC-2001_1x2032
- moved C6 17.0 mm to (87.0, 97.0), turned to 90 degrees
- moved U1 10.3 mm to (91.0, 97.0), turned to 90 degrees
- moved U2 5.65 mm to (101.9, 91.7), turned to -90 degrees
- moved R4 5.49 mm to (94.6, 97.0), turned to -90 degrees
- moved R3 4.16 mm to (90.0, 92.4), turned to 0 degrees
- moved C1 3.58 mm to (100.2, 89.6), turned to -90 degrees
- moved C2 3.42 mm to (106.6, 89.6), turned to -90 degrees
- moved BT1 1.00 mm to (100.0, 110.0), turned to 0 degrees
- turned SW1 to 0 degrees
Routing:
- net D+: track 8.66 -> 15.2 mm
- net VDD: track 6.54 -> 0.31 mm
- net SWIO: track 5.78 -> 10.8 mm
- net D-: track 12.1 -> 15.8 mm
- net KEY: track 15.6 -> 15.5 mm, vias 0 -> 1
- net GND: vias 6 -> 43
- net BAT: vias 4 -> 8
- added copper zone on B.Cu, net VDD
Other:
- board text added: "0u1"
- board text added: "10k"
- board text added: "1k5"
- board text added: "1u"
- board text added: "3V3"
- board text added: "4k7"
- board text added: "AP7333"
- board text added: "BAT"
- board text added: "CR2032"
- board text added: "GND"
- board text added: "SWIO"
- board text added: "VDD"
- board text added: "ueckoken.club"
